Commit message: wip: resolving collision checks

File: grasping_description/urdf/ur10-two-finger.urdf.xacro (robot description, xacro)
@@ -110,13 +110,13 @@
 		parent="$(arg tf_prefix)tool0"
 		prefix="$(arg tf_prefix)"
-		xyz="0 0 0.008"
-		rpy="0 0 0" />
+		xyz="0 0 0"
+		rpy="0 0 -1.57" />
 	<xacro:two_finger_gripper
 		parent="$(arg tf_prefix)camera_mount_link"
 		prefix="$(arg tf_prefix)"
-		xyz="0 0 0"
+		xyz="0 0 0.008"
 		rpy="0 0 1.57" />
 	<xacro:sensor_d435 parent="$(arg tf_prefix)camera_mount_link" name="$(arg tf_prefix)camera">
-		<origin xyz="-0.085 0 0.035" rpy="0 -1.57 0" />
+		<origin xyz="-0.085 0 0.043" rpy="0 -1.57 0" />
 	</xacro:sensor_d435>
 	<xacro:if value="$(arg sim_gazebo)">

File: grasping_description/xacro/camera-mount.urdf.xacro (robot description, xacro)
@@ -7,5 +7,5 @@
 		<link name="${prefix}camera_mount_link">
 			<visual>
-				<origin xyz="0 0 0" rpy="-1.57 3.14 1.57" />
+				<origin xyz="0 0 0.008" rpy="1.57 0 -1.57" />
 				<geometry>
 					<mesh filename="package://grasping_description/meshes/camera-mount.stl" scale="${scale}" />
@@ -14,7 +14,7 @@
 			</visual>
 			<collision>
-				<origin xyz="0 0 0" rpy="-1.57 3.14 1.57" />
+				<origin xyz="0 0 0.008" rpy="1.57 0 -1.57" />
 				<geometry>
-					<mesh filename="package://grasping_description/meshes/camera-mount.stl" scale="${scale}" />
+					<mesh filename="package://grasping_description/meshes/camera-mount.stl" scale="0.95 0.95 0.95" />
 				</geometry>
 			</collision>
