Commit message: fixed issues with demo hardware launch file and added documentation

File: grasping_description/xacro/camera/camera-mount.urdf.xacro (robot description, xacro)
@@ -9,5 +9,5 @@
 				<origin xyz="0 0 0.008" rpy="1.57 0 -1.57" />
 				<geometry>
-					<mesh filename="package://grasping_description/meshes/camera-mount.stl" scale="${scale}" />
+					<mesh filename="package://grasping_description/meshes/camera/camera-mount.stl" scale="${scale}" />
 				</geometry>
 				<material name="${prefix}camera_mount_gray" />
@@ -16,5 +16,5 @@
 				<origin xyz="0 0 0.008" rpy="1.57 0 -1.57" />
 				<geometry>
-					<mesh filename="package://grasping_description/meshes/camera-mount.stl" scale="0.95 0.95 0.95" />
+					<mesh filename="package://grasping_description/meshes/camera/camera-mount.stl" scale="0.95 0.95 0.95" />
 				</geometry>
 			</collision>

File: grasping_description/xacro/ur10_soft_two_fingers/ur10-soft-two-fingers.urdf.xacro (robot description, xacro)
@@ -3,5 +3,5 @@
 	<xacro:arg name="name" default="ur"/>
 	<xacro:include filename="$(find ur_description)/urdf/ur_macro.xacro"/>
-	<xacro:include filename="$(find grasping_description)/xacro/camera-mount.urdf.xacro"/>
+	<xacro:include filename="$(find grasping_description)/xacro/camera/camera-mount.urdf.xacro"/>
 	<xacro:include filename="$(find gripper_description)/xacro/two-finger-gripper.urdf.xacro"/>
 	<xacro:include filename="$(find realsense2_description)/urdf/_d435.urdf.xacro"/>
@@ -12,4 +12,5 @@
 	<xacro:arg name="physical_params" default="$(find ur_description)/config/$(arg ur_type)/physical_parameters.yaml"/>
 	<xacro:arg name="visual_params" default="$(find ur_description)/config/$(arg ur_type)/visual_parameters.yaml"/>
+	<xacro:arg name="generate_ros2_control_tag" default="true"/>
 	<xacro:arg name="transmission_hw_interface" default=""/>
 	<xacro:arg name="safety_limits" default="false"/>
@@ -40,6 +41,4 @@
 	<xacro:arg name="sim_ignition" default="false" />
 	<xacro:arg name="simulation_controllers" default="" />
-	<xacro:arg name="initial_positions_file" default="$(find ur_description)/config/initial_positions.yaml"/>
-	<xacro:property name="initial_positions_file" default="$(arg initial_positions_file)"/>
 	<xacro:property name="is_sim_gazebo" value="$(arg sim_gazebo)"/>
 	<xacro:property name="is_sim_ignition" value="$(arg sim_ignition)"/>
@@ -77,4 +76,5 @@
 		physical_parameters_file="$(arg physical_params)"
 		visual_parameters_file="$(arg visual_params)"
+		generate_ros2_control_tag="$(arg generate_ros2_control_tag)"
 		transmission_hw_interface="$(arg transmission_hw_interface)"
 		safety_limits="$(arg safety_limits)"
@@ -86,5 +86,4 @@
 		sim_ignition="$(arg sim_ignition)"
 		headless_mode="$(arg headless_mode)"
-		initial_positions="${xacro.load_yaml(initial_positions_file)}"
 		use_tool_communication="$(arg use_tool_communication)"
 		tool_voltage="$(arg tool_voltage)"

File: grasping_moveit_config/ur10_soft_two_fingers_moveit_config/config/ur.ros2_control.xacro (robot description, xacro)
@@ -2,5 +2,5 @@
 <robot xmlns:xacro="http://www.ros.org/wiki/xacro">
     <xacro:macro name="ur_ros2_control" params="name initial_positions_file">
-        <xacro:property name="initial_positions" value="${load_yaml(initial_positions_file)['initial_positions']}"/>
+        <xacro:property name="initial_positions" value="${xacro.load_yaml(initial_positions_file)['initial_positions']}"/>
         <ros2_control name="${name}" type="system">
             <hardware>
@@ -8,46 +8,58 @@
                 <plugin>mock_components/GenericSystem</plugin>
             </hardware>
-            <joint name="shoulder_pan_joint">
-                <command_interface name="position"/>
-                <state_interface name="position">
-                  <param name="initial_value">${initial_positions['shoulder_pan_joint']}</param>
-                </state_interface>
-                <state_interface name="velocity"/>
-            </joint>
-            <joint name="shoulder_lift_joint">
-                <command_interface name="position"/>
-                <state_interface name="position">
-                  <param name="initial_value">${initial_positions['shoulder_lift_joint']}</param>
-                </state_interface>
-                <state_interface name="velocity"/>
-            </joint>
-            <joint name="elbow_joint">
-                <command_interface name="position"/>
-                <state_interface name="position">
-                  <param name="initial_value">${initial_positions['elbow_joint']}</param>
-                </state_interface>
-                <state_interface name="velocity"/>
-            </joint>
-            <joint name="wrist_1_joint">
-                <command_interface name="position"/>
-                <state_interface name="position">
-                  <param name="initial_value">${initial_positions['wrist_1_joint']}</param>
-                </state_interface>
-                <state_interface name="velocity"/>
-            </joint>
-            <joint name="wrist_2_joint">
-                <command_interface name="position"/>
-                <state_interface name="position">
-                  <param name="initial_value">${initial_positions['wrist_2_joint']}</param>
-                </state_interface>
-                <state_interface name="velocity"/>
-            </joint>
-            <joint name="wrist_3_joint">
-                <command_interface name="position"/>
-                <state_interface name="position">
-                  <param name="initial_value">${initial_positions['wrist_3_joint']}</param>
-                </state_interface>
-                <state_interface name="velocity"/>
-            </joint>
+                        <joint name="shoulder_pan_joint">
+                                <command_interface name="position"/>
+                                <state_interface name="position">
+                                    <param name="initial_value">${initial_positions['shoulder_pan_joint']}</param>
+                                </state_interface>
+                                <state_interface name="velocity">
+                                    <param name="initial_value">0.0</param>
+                                </state_interface>
+                        </joint>
+                        <joint name="shoulder_lift_joint">
+                                <command_interface name="position"/>
+                                <state_interface name="position">
+                                    <param name="initial_value">${initial_positions['shoulder_lift_joint']}</param>
+                                </state_interface>
+                                <state_interface name="velocity">
+                                    <param name="initial_value">0.0</param>
+                                </state_interface>
+                        </joint>
+                        <joint name="elbow_joint">
+                                <command_interface name="position"/>
+                                <state_interface name="position">
+                                    <param name="initial_value">${initial_positions['elbow_joint']}</param>
+                                </state_interface>
+                                <state_interface name="velocity">
+                                    <param name="initial_value">0.0</param>
+                                </state_interface>
+                        </joint>
+                        <joint name="wrist_1_joint">
+                                <command_interface name="position"/>
+                                <state_interface name="position">
+                                    <param name="initial_value">${initial_positions['wrist_1_joint']}</param>
+                                </state_interface>
+                                <state_interface name="velocity">
+                                    <param name="initial_value">0.0</param>
+                                </state_interface>
+                        </joint>
+                        <joint name="wrist_2_joint">
+                                <command_interface name="position"/>
+                                <state_interface name="position">
+                                    <param name="initial_value">${initial_positions['wrist_2_joint']}</param>
+                                </state_interface>
+                                <state_interface name="velocity">
+                                    <param name="initial_value">0.0</param>
+                                </state_interface>
+                        </joint>
+                        <joint name="wrist_3_joint">
+                                <command_interface name="position"/>
+                                <state_interface name="position">
+                                    <param name="initial_value">${initial_positions['wrist_3_joint']}</param>
+                                </state_interface>
+                                <state_interface name="velocity">
+                                    <param name="initial_value">0.0</param>
+                                </state_interface>
+                        </joint>
             <joint name="gripper_planar_5">
                 <command_interface name="position"/>
@@ -55,5 +67,7 @@
                   <param name="initial_value">${initial_positions['gripper_planar_5']}</param>
                 </state_interface>
-                <state_interface name="velocity"/>
+                                <state_interface name="velocity">
+                                    <param name="initial_value">0.0</param>
+                                </state_interface>
             </joint>
             <joint name="gripper_planar_4">
@@ -62,5 +76,7 @@
                   <param name="initial_value">${initial_positions['gripper_planar_4']}</param>
                 </state_interface>
-                <state_interface name="velocity"/>
+                                <state_interface name="velocity">
+                                    <param name="initial_value">0.0</param>
+                                </state_interface>
             </joint>
         </ros2_control>

File: grasping_moveit_config/ur10_soft_two_fingers_moveit_config/config/ur.urdf.xacro (robot description, xacro)
@@ -3,5 +3,5 @@
     <xacro:arg name="initial_positions_file" default="initial_positions.yaml" />
     <!-- Import ur urdf file -->
-    <xacro:include filename="$(find grasping_description)/xacro/ur10-soft-two-fingers.urdf.xacro" />
+    <xacro:include filename="$(find grasping_description)/xacro/ur10_soft_two_fingers/ur10-soft-two-fingers.urdf.xacro" />
     <!-- Import control_xacro -->
     <xacro:include filename="ur.ros2_control.xacro" />

Commit message: added robot base. tested with demo. pending test on hardware_with_moveit

File: grasping_description/xacro/camera/camera-mount.urdf.xacro (robot description, xacro)
@@ -16,5 +16,5 @@
 				<origin xyz="0 0 0.008" rpy="1.57 0 -1.57" />
 				<geometry>
-					<mesh filename="package://grasping_description/meshes/camera/camera-mount.stl" scale="0.95 0.95 0.95" />
+					<mesh filename="package://grasping_description/meshes/camera/camera-mount.stl" scale="${scale}" />
 				</geometry>
 			</collision>

File: grasping_description/xacro/ur10_soft_two_fingers/ur10-soft-two-fingers.urdf.xacro (robot description, xacro)
@@ -3,4 +3,5 @@
 	<xacro:arg name="name" default="ur"/>
 	<xacro:include filename="$(find ur_description)/urdf/ur_macro.xacro"/>
+	<xacro:include filename="$(find grasping_description)/xacro/robot-base/ur10-base.urdf.xacro"/>
 	<xacro:include filename="$(find grasping_description)/xacro/camera/camera-mount.urdf.xacro"/>
 	<xacro:include filename="$(find gripper_description)/xacro/two-finger-gripper.urdf.xacro"/>
@@ -68,8 +69,13 @@
 		</joint>
 	</xacro:if>
+	<xacro:ur10_base
+		parent="world"
+		prefix="$(arg tf_prefix)"
+		xyz="0 0 0.865"
+		rpy="0 0 0" />
 	<xacro:ur_robot
 		name="$(arg name)"
 		tf_prefix="$(arg tf_prefix)"
-		parent="world"
+		parent="$(arg tf_prefix)ur10_base_link"
 		joint_limits_parameters_file="$(arg joint_limit_params)"
 		kinematics_parameters_file="$(arg kinematics_params)"

File: grasping_moveit_config/ur10_soft_two_fingers_moveit_config/config/ur.ros2_control.xacro (robot description, xacro)
@@ -2,5 +2,5 @@
 <robot xmlns:xacro="http://www.ros.org/wiki/xacro">
     <xacro:macro name="ur_ros2_control" params="name initial_positions_file">
-        <xacro:property name="initial_positions" value="${xacro.load_yaml(initial_positions_file)['initial_positions']}"/>
+    <xacro:property name="initial_positions" value="${xacro.load_yaml(initial_positions_file)['initial_positions']}"/>
         <ros2_control name="${name}" type="system">
             <hardware>
@@ -8,58 +8,58 @@
                 <plugin>mock_components/GenericSystem</plugin>
             </hardware>
-                        <joint name="shoulder_pan_joint">
-                                <command_interface name="position"/>
-                                <state_interface name="position">
-                                    <param name="initial_value">${initial_positions['shoulder_pan_joint']}</param>
-                                </state_interface>
-                                <state_interface name="velocity">
-                                    <param name="initial_value">0.0</param>
-                                </state_interface>
-                        </joint>
-                        <joint name="shoulder_lift_joint">
-                                <command_interface name="position"/>
-                                <state_interface name="position">
-                                    <param name="initial_value">${initial_positions['shoulder_lift_joint']}</param>
-                                </state_interface>
-                                <state_interface name="velocity">
-                                    <param name="initial_value">0.0</param>
-                                </state_interface>
-                        </joint>
-                        <joint name="elbow_joint">
-                                <command_interface name="position"/>
-                                <state_interface name="position">
-                                    <param name="initial_value">${initial_positions['elbow_joint']}</param>
-                                </state_interface>
-                                <state_interface name="velocity">
-                                    <param name="initial_value">0.0</param>
-                                </state_interface>
-                        </joint>
-                        <joint name="wrist_1_joint">
-                                <command_interface name="position"/>
-                                <state_interface name="position">
-                                    <param name="initial_value">${initial_positions['wrist_1_joint']}</param>
-                                </state_interface>
-                                <state_interface name="velocity">
-                                    <param name="initial_value">0.0</param>
-                                </state_interface>
-                        </joint>
-                        <joint name="wrist_2_joint">
-                                <command_interface name="position"/>
-                                <state_interface name="position">
-                                    <param name="initial_value">${initial_positions['wrist_2_joint']}</param>
-                                </state_interface>
-                                <state_interface name="velocity">
-                                    <param name="initial_value">0.0</param>
-                                </state_interface>
-                        </joint>
-                        <joint name="wrist_3_joint">
-                                <command_interface name="position"/>
-                                <state_interface name="position">
-                                    <param name="initial_value">${initial_positions['wrist_3_joint']}</param>
-                                </state_interface>
-                                <state_interface name="velocity">
-                                    <param name="initial_value">0.0</param>
-                                </state_interface>
-                        </joint>
+            <joint name="shoulder_pan_joint">
+                <command_interface name="position"/>
+                <state_interface name="position">
+                  <param name="initial_value">${initial_positions['shoulder_pan_joint']}</param>
+                </state_interface>
+                <state_interface name="velocity">
+                  <param name="initial_value">0.0</param>
+                </state_interface>
+            </joint>
+            <joint name="shoulder_lift_joint">
+                <command_interface name="position"/>
+                <state_interface name="position">
+                  <param name="initial_value">${initial_positions['shoulder_lift_joint']}</param>
+                </state_interface>
+                <state_interface name="velocity">
+                  <param name="initial_value">0.0</param>
+                </state_interface>
+            </joint>
+            <joint name="elbow_joint">
+                <command_interface name="position"/>
+                <state_interface name="position">
+                  <param name="initial_value">${initial_positions['elbow_joint']}</param>
+                </state_interface>
+                <state_interface name="velocity">
+                  <param name="initial_value">0.0</param>
+                </state_interface>
+            </joint>
+            <joint name="wrist_1_joint">
+                <command_interface name="position"/>
+                <state_interface name="position">
+                  <param name="initial_value">${initial_positions['wrist_1_joint']}</param>
+                </state_interface>
+                <state_interface name="velocity">
+                  <param name="initial_value">0.0</param>
+                </state_interface>
+            </joint>
+            <joint name="wrist_2_joint">
+                <command_interface name="position"/>
+                <state_interface name="position">
+                  <param name="initial_value">${initial_positions['wrist_2_joint']}</param>
+                </state_interface>
+                <state_interface name="velocity">
+                  <param name="initial_value">0.0</param>
+                </state_interface>
+            </joint>
+            <joint name="wrist_3_joint">
+                <command_interface name="position"/>
+                <state_interface name="position">
+                  <param name="initial_value">${initial_positions['wrist_3_joint']}</param>
+                </state_interface>
+                <state_interface name="velocity">
+                  <param name="initial_value">0.0</param>
+                </state_interface>
+            </joint>
             <joint name="gripper_planar_5">
                 <command_interface name="position"/>
@@ -67,7 +67,7 @@
                   <param name="initial_value">${initial_positions['gripper_planar_5']}</param>
                 </state_interface>
-                                <state_interface name="velocity">
-                                    <param name="initial_value">0.0</param>
-                                </state_interface>
+                <state_interface name="velocity">
+                  <param name="initial_value">0.0</param>
+                </state_interface>
             </joint>
             <joint name="gripper_planar_4">
@@ -76,7 +76,7 @@
                   <param name="initial_value">${initial_positions['gripper_planar_4']}</param>
                 </state_interface>
-                                <state_interface name="velocity">
-                                    <param name="initial_value">0.0</param>
-                                </state_interface>
+                <state_interface name="velocity">
+                  <param name="initial_value">0.0</param>
+                </state_interface>
             </joint>
         </ros2_control>

Commit message: added use_demo launch parameter

File: grasping_description/xacro/camera/camera-mount.urdf.xacro (robot description, xacro)
@@ -7,5 +7,5 @@
 		<link name="${prefix}camera_mount_link">
 			<visual>
-				<origin xyz="0 0 0.008" rpy="1.57 0 -1.57" />
+				<origin xyz="0 0 0.008" rpy="1.57 0 1.57" />
 				<geometry>
 					<mesh filename="package://grasping_description/meshes/camera/camera-mount.stl" scale="${scale}" />
@@ -14,5 +14,5 @@
 			</visual>
 			<collision>
-				<origin xyz="0 0 0.008" rpy="1.57 0 -1.57" />
+				<origin xyz="0 0 0.008" rpy="1.57 0 1.57" />
 				<geometry>
 					<mesh filename="package://grasping_description/meshes/camera/camera-mount.stl" scale="${scale}" />

File: grasping_description/xacro/ur10_soft_two_fingers/ur10-soft-two-fingers.urdf.xacro (robot description, xacro)
@@ -116,5 +116,5 @@
 		prefix="$(arg tf_prefix)"
 		xyz="0 0 0"
-		rpy="0 0 -1.57" />
+		rpy="0 0 0" />
 	<xacro:two_finger_gripper
 		parent="$(arg tf_prefix)camera_mount_link"

Commit message: fixed issues in the tf which conflicted with hardware

File: grasping_description/xacro/camera/camera-mount.urdf.xacro (robot description, xacro)
@@ -7,5 +7,5 @@
 		<link name="${prefix}camera_mount_link">
 			<visual>
-				<origin xyz="0 0 0.008" rpy="1.57 0 1.57" />
+				<origin xyz="0 0 0.008" rpy="1.57 0 0" />
 				<geometry>
 					<mesh filename="package://grasping_description/meshes/camera/camera-mount.stl" scale="${scale}" />
@@ -14,5 +14,5 @@
 			</visual>
 			<collision>
-				<origin xyz="0 0 0.008" rpy="1.57 0 1.57" />
+				<origin xyz="0 0 0.008" rpy="1.57 0 0" />
 				<geometry>
 					<mesh filename="package://grasping_description/meshes/camera/camera-mount.stl" scale="${scale}" />

File: grasping_description/xacro/ur10_soft_two_fingers/ur10-soft-two-fingers.urdf.xacro (robot description, xacro)
@@ -121,7 +121,7 @@
 		prefix="$(arg tf_prefix)"
 		xyz="0 0 0.008"
-		rpy="0 0 1.57" />
+		rpy="0 0 0" />
 	<xacro:sensor_d435 parent="$(arg tf_prefix)camera_mount_link" name="$(arg tf_prefix)camera">
-		<origin xyz="-0.085 0 0.043" rpy="0 -1.57 0" />
+		<origin xyz="0 -0.085 0.043" rpy="0 -1.57 1.57" />
 	</xacro:sensor_d435>
 	<xacro:if value="$(arg sim_gazebo)">
