Commit message: added tm12s models, moveit config, launch files and documentation

File: grasping_description/xacro/tm12s_soft_two_fingers/tm12s-soft-tiw-fingers.urdf.xacro (robot description, xacro)
@@ -17,5 +17,5 @@
 		rpy="0 0 0" />
 	<joint name="$(arg prefix)robot_base_to_tm12s_base" type="fixed">
-		<origin xyz="0 0 0" rpy="0 0 0" />
+		<origin xyz="0 0 0" rpy="0 0 0.785" />
 		<parent link="$(arg prefix)tm12s_base_link" />
 		<child link="$(arg prefix)base" />
