Commit message: fixed tm12s robot base description

File: grasping_description/xacro/robot-base/tm12s-base.urdf.xacro (robot description, xacro)
@@ -7,5 +7,5 @@
 		<link name="${prefix}tm12s_base_link">
 			<visual>
-				<origin xyz="0 0 0" rpy="0 3.14 0" />
+				<origin xyz="0 0 0" rpy="0 3.14 0.785" />
 				<geometry>
 					<mesh filename="package://grasping_description/meshes/robot-base/tm12s-base.stl" scale="${scale}" />
@@ -14,5 +14,5 @@
 			</visual>
 			<collision>
-				<origin xyz="0 0 0" rpy="0 3.14 0" />
+				<origin xyz="0 0 0" rpy="0 3.14 0.785" />
 				<geometry>
 					<mesh filename="package://grasping_description/meshes/robot-base/tm12s-base.stl" scale="${scale}" />
